File: Ponte_H_L293E.sch (EAGLE design)
At the start: 0 parts

Commit message: schematico L293E+BT
Parts:
- added C1, C4: 10uF / 16V, rcl_LargePads:CPOL-EUE5-8.5
- added C2, C3: 100nF, rcl_LargePads:C-EU050-025X075
- added D1, D2, D3, D4: 1N4004, diode_LargePads:1N4004
- added IC1: L293EDIL20, L293:L293EDIL20
- added IC2: 74HC14N, 74xx-eu:74HC14N
- added IC3: 7805, v-reg_LargePads:78XXS
- added JP1: (no value), pinhead:PINHD-1X6
- added OK1, OK2: TIL191, optocoupler:TIL191
- added R1, R3: 180, rcl_LargePads:R-EU_0207/10
- added R2, R4: 2.2k, rcl_LargePads:R-EU_0207/10
- added R5: 1.8k, rcl_LargePads:R-EU_0207/10
- added R6: 3.3k, rcl_LargePads:R-EU_0207/10
- added R7: 1.2k, rcl_LargePads:R-EU_0207/10
- added U1: HC05, HC05_HC06:HC05
- added X1, X2: (no value), con-ptr500:AK500/2
Connections:
- new net +5V: C1.+, C2.1, C3.1, IC1.VSS, IC2P.VCC, IC3.OUT, R2.2, R4.2
- new net +9V: C4.+, D1.C, D3.C, IC1.VS, IC3.IN, X2-2.KL
- new net 1Y: D3.A, D4.C, IC1.OUT1, X1-2.KL
- new net 2Y: D1.A, D2.C, IC1.OUT2, X1-1.KL
- new net GND: C1.-, C2.2, C3.2, C4.-, D2.A, D4.A, IC1.CE2, IC1.GND1, IC1.GND2, IC1.GND3, IC1.GND4, IC1.IN3, IC1.IN4, IC1.SENSE1, IC1.SENSE2, IC1.SENSE3, IC1.SENSE4, IC2P.GND, IC3.GND, OK1.EMIT, OK2.EMIT, X2-1.KL
- new net GNDA: JP1.6, OK1.C, OK2.C, R6.1, U1.GND
- new net I/!A!: JP1.5, R3.1
- new net N$1: IC1.CE1, IC2A.O
- new net N$11: IC2A.I, OK1.COL, R2.1
- new net N$13: R5.2, R6.2, U1.RXD
- new net N$2: IC1.IN1, IC2B.I, OK2.COL, R4.1
- new net N$3: OK2.A, R3.2
- new net N$4: IC1.IN2, IC2B.O
- new net N$5: OK1.A, R1.2
- new net N$6: R7.2, U1.TXD
- new net PWM: JP1.4, R1.1
- new net RX_5V: JP1.3, R7.1
- new net TX_5V: JP1.2, R5.1
- new net VCC: JP1.1, U1.VCC
Other:
- note added: "+5V Arduino"
- note added: "+9V Alimentazione motori"
- note added: "Comando velocità e Avanti/Indietro per un motore in corrente continua"
- note added: "Dominio di alimentazione di Arduino (con i 5V e la massa GNDA di Arduno)"
- note added: "GND microcontrollore"
- note added: "IND/!AV! M1"
- note added: "Modulo Bluetooth"
- note added: "Motore DC 1"
- note added: "ON/!OFF! o PWM M1"
- note added: "RX Arduino <-"
- note added: "TX Arduino ->"
