File: Ponte_H_L293E.brd (EAGLE design)
At the start: 50 x 80 mm, 24 parts, among them IC1 L293EDIL20, IC2 74HC14N, IC3 7805, U1 HC05

Commit message: creato pdf schematico
Parts:
- moved C1 1.27 mm to (41.9, 33.0)
Routing:
- net GND: track 195.8 -> 196.9 mm
- net +5V: track 53.7 -> 54.5 mm
Other:
- board text added: "DL23"
Changed lines of the file:
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@@
 <text x="2.54" y="22.86" size="2.1844" layer="1" font="vector" ratio="15">+Vcc</text>
 <text x="3.81" y="3.81" size="2.1844" layer="1" font="vector" ratio="15">GNDA</text>
+<text x="39.37" y="76.2" size="2.1844" layer="16" font="vector" ratio="20" rot="MR0" align="center">DL23</text>
+<text x="7.62" y="24.13" size="2.1844" layer="16" font="vector" ratio="20" rot="MR0" align="center">DL23</text>
 </plain>
 <attributes>
@@
 </autorouter>
 <elements>
-<element name="C1" library="rcl_LargePads" package="E5-8,5" value="10uF / 16V" x="43.18" y="33.02" smashed="yes">
-<attribute name="NAME" x="47.3202" y="35.306" size="1.27" layer="25" ratio="10"/>
-<attribute name="VALUE" x="40.6654" y="29.9974" size="1.27" layer="27" ratio="10"/>
+<element name="C1" library="rcl_LargePads" package="E5-8,5" value="10uF / 16V" x="41.91" y="33.02" smashed="yes">
+<attribute name="NAME" x="46.0502" y="35.306" size="1.27" layer="25" ratio="10"/>
+<attribute name="VALUE" x="39.3954" y="29.9974" size="1.27" layer="27" ratio="10"/>
 </element>
 <element name="C2" library="rcl_LargePads" package="C050-025X075" value="100nF" x="38.1" y="45.72" smashed="yes" rot="R90">
@@
 <wire x1="44.45" y1="22.86" x2="45.72" y2="24.13" width="0.8" layer="1"/>
 <via x="45.72" y="24.13" extent="1-16" drill="0.8" diameter="2"/>
-<wire x1="45.72" y1="24.13" x2="45.72" y2="33.02" width="0.8" layer="16"/>
+<wire x1="44.45" y1="33.02" x2="45.72" y2="31.75" width="0.8" layer="16"/>
+<wire x1="45.72" y1="31.75" x2="45.72" y2="24.13" width="0.8" layer="16"/>
 <wire x1="35.56" y1="7.62" x2="35.56" y2="11.43" width="0.8" layer="16"/>
 <wire x1="43.18" y1="48.26" x2="41.91" y2="48.26" width="1.27" layer="16"/>
@@
 <wire x1="43.18" y1="48.26" x2="46.99" y2="48.26" width="1.2" layer="16"/>
 <wire x1="46.99" y1="48.26" x2="46.99" y2="38.1" width="1.2" layer="16"/>
-<wire x1="46.99" y1="38.1" x2="45.72" y2="36.83" width="1.2" layer="16"/>
-<wire x1="45.72" y1="36.83" x2="45.72" y2="33.02" width="1.2" layer="16"/>
+<wire x1="46.99" y1="38.1" x2="44.45" y2="35.56" width="1.2" layer="16"/>
+<wire x1="44.45" y1="35.56" x2="44.45" y2="33.02" width="1.2" layer="16"/>
 <wire x1="46.99" y1="55.88" x2="44.45" y2="58.42" width="1.2" layer="16"/>
 <wire x1="44.45" y1="58.42" x2="44.45" y2="67.31" width="1.2" layer="16"/>
@@
 <wire x1="26.67" y1="29.21" x2="27.94" y2="30.48" width="0.8" layer="16"/>
 <wire x1="29.21" y1="43.18" x2="38.1" y2="43.18" width="0.8" layer="16"/>
-<wire x1="41.91" y1="39.37" x2="38.1" y2="43.18" width="0.8" layer="16"/>
-<wire x1="41.91" y1="26.67" x2="40.64" y2="27.94" width="0.8" layer="16"/>
-<wire x1="40.64" y1="27.94" x2="40.64" y2="30.48" width="0.8" layer="16"/>
-<wire x1="40.64" y1="30.48" x2="40.64" y2="33.02" width="0.8" layer="16"/>
-<wire x1="40.64" y1="33.02" x2="40.64" y2="38.1" width="0.8" layer="16"/>
-<wire x1="40.64" y1="38.1" x2="41.91" y2="39.37" width="0.8" layer="16"/>
-<wire x1="27.94" y1="30.48" x2="40.64" y2="30.48" width="0.8" layer="16"/>
+<wire x1="40.64" y1="39.37" x2="38.1" y2="41.91" width="0.8" layer="16"/>
+<wire x1="38.1" y1="41.91" x2="38.1" y2="43.18" width="0.8" layer="16"/>
+<wire x1="41.91" y1="26.67" x2="40.64" y2="26.67" width="0.8" layer="16"/>
+<wire x1="40.64" y1="26.67" x2="39.37" y2="27.94" width="0.8" layer="16"/>
+<wire x1="39.37" y1="27.94" x2="39.37" y2="30.48" width="0.8" layer="16"/>
+<wire x1="39.37" y1="30.48" x2="39.37" y2="33.02" width="0.8" layer="16"/>
+<wire x1="39.37" y1="33.02" x2="39.37" y2="38.1" width="0.8" layer="16"/>
+<wire x1="40.64" y1="39.37" x2="41.91" y2="39.37" width="0.8" layer="16"/>
+<wire x1="40.64" y1="39.37" x2="39.37" y2="38.1" width="0.8" layer="16"/>
+<wire x1="27.94" y1="30.48" x2="39.37" y2="30.48" width="0.8" layer="16"/>
 </signal>
 <signal name="+9V" class="2">
@@
 <contactref element="U1" pad="4"/>
 <contactref element="R7" pad="2"/>
-<wire x1="43.18" y1="15.24" x2="38.1" y2="15.24" width="0.8" layer="16"/>
-<wire x1="35.56" y1="17.78" x2="31.75" y2="17.78" width="0.8" layer="16"/>
-<wire x1="38.1" y1="15.24" x2="35.56" y2="17.78" width="0.8" layer="16"/>
+<wire x1="43.18" y1="15.24" x2="36.83" y2="15.24" width="0.8" layer="16"/>
+<wire x1="34.29" y1="17.78" x2="31.75" y2="17.78" width="0.8" layer="16"/>
+<wire x1="36.83" y1="15.24" x2="34.29" y2="17.78" width="0.8" layer="16"/>
 </signal>
 </signals>
